File: vcu.brd (EAGLE design)
At the start: 44.4 x 48 mm, 31 parts, among them IC1 7805DT, IC2 MCP2551/SN, U1 ATMEGA328P-AU, U2 PMIC-LDO-XC6206P332MR-G(SOT23)

Commit message: improvement
Parts:
- moved C3 0.73 mm to (38.6, 56.9), turned to 270 degrees
Connections:
- removed net N$1: C3.2, JP7.1
- removed net VSS: U2.1
- net GND: now also C3.2, JP7.1, U2.1
Routing:
- net GND: track 205.3 -> 219.7 mm, vias 3 -> 4
- net ADC7: track 45.2 -> 39.3 mm, vias 2 -> 4
- net B3/MOSI: track 41.1 -> 36.0 mm
- net N$1: track 4.44 -> 0.00 mm
- net N$2: track 23.1 -> 21.7 mm
- net B5/SCK: track 122.4 -> 123.2 mm
- net D1: track 25.0 -> 25.6 mm
Other:
- board text added: "Ampersand VCU"
- board text added: "Rev 1.0"
