File: vcu.sch (EAGLE design)
At the start: 31 parts, among them IC1 7805DT, IC2 MCP2551/SN, U1 ATMEGA328P-AU, U2 PMIC-LDO-XC6206P332MR-G(SOT23)

Commit message: improvement
Connections:
- removed net N$1: C3.2, JP7.1
- removed net VSS: U2.VSS
- net GND: now also C3.2, JP7.1, U2.VSS
Changed lines of the file:
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@@
 <part name="IC2" library="microchip-dspic" deviceset="MCP2551" device="/SN"/>
 <part name="P+2" library="supply1" library_urn="urn:adsk.eagle:library:371" deviceset="+5V" device=""/>
-<part name="GND2" library="supply1" library_urn="urn:adsk.eagle:library:371" deviceset="GND" device=""/>
 <part name="GND3" library="supply1" library_urn="urn:adsk.eagle:library:371" deviceset="GND" device=""/>
 <part name="GND4" library="supply1" library_urn="urn:adsk.eagle:library:371" deviceset="GND" device=""/>
@@
 <part name="+3V1" library="supply1" library_urn="urn:adsk.eagle:library:371" deviceset="+3V3" device=""/>
 <part name="+3V2" library="supply1" library_urn="urn:adsk.eagle:library:371" deviceset="+3V3" device=""/>
-<part name="GND14" library="supply1" library_urn="urn:adsk.eagle:library:371" deviceset="GND" device=""/>
 <part name="GND15" library="supply1" library_urn="urn:adsk.eagle:library:371" deviceset="GND" device=""/>
 <part name="JP8" library="pinhead" library_urn="urn:adsk.eagle:library:325" deviceset="PINHD-1X10" device="" package3d_urn="urn:adsk.eagle:package:22406/2"/>
@@
 <part name="GND16" library="supply1" library_urn="urn:adsk.eagle:library:371" deviceset="GND" device=""/>
 <part name="IC1" library="linear" library_urn="urn:adsk.eagle:library:262" deviceset="78*" device="DT" package3d_urn="urn:adsk.eagle:package:16415/2" technology="05"/>
+<part name="GND2" library="supply1" library_urn="urn:adsk.eagle:library:371" deviceset="GND" device=""/>
+<part name="GND12" library="supply1" library_urn="urn:adsk.eagle:library:371" deviceset="GND" device=""/>
 </parts>
 <sheets>
@@
 <attribute name="VALUE" x="2.54" y="109.22" size="1.778" layer="96" rot="R90"/>
 </instance>
-<instance part="GND2" gate="1" x="-35.56" y="83.82" smashed="yes">
-<attribute name="VALUE" x="-38.1" y="81.28" size="1.778" layer="96"/>
-</instance>
-<instance part="GND3" gate="1" x="2.54" y="86.36" smashed="yes">
-<attribute name="VALUE" x="0" y="83.82" size="1.778" layer="96"/>
+<instance part="GND3" gate="1" x="2.54" y="83.82" smashed="yes">
+<attribute name="VALUE" x="0" y="81.28" size="1.778" layer="96"/>
 </instance>
 <instance part="GND4" gate="1" x="-15.24" y="83.82" smashed="yes">
@@
 <attribute name="VALUE" x="195.58" y="-7.62" size="1.778" layer="96" rot="R90"/>
 </instance>
-<instance part="GND14" gate="1" x="106.68" y="-33.02" smashed="yes">
-<attribute name="VALUE" x="104.14" y="-35.56" size="1.778" layer="96"/>
-</instance>
 <instance part="GND15" gate="1" x="195.58" y="2.54" smashed="yes">
 <attribute name="VALUE" x="193.04" y="0" size="1.778" layer="96"/>
@@
 <attribute name="NAME" x="-22.86" y="109.855" size="1.778" layer="95"/>
 <attribute name="VALUE" x="-22.86" y="107.315" size="1.778" layer="96"/>
+</instance>
+<instance part="GND2" gate="1" x="-35.56" y="83.82" smashed="yes">
+<attribute name="VALUE" x="-38.1" y="81.28" size="1.778" layer="96"/>
+</instance>
+<instance part="GND12" gate="1" x="106.68" y="-35.56" smashed="yes">
+<attribute name="VALUE" x="104.14" y="-38.1" size="1.778" layer="96"/>
 </instance>
 </instances>
@@
 <pinref part="C2" gate="G$1" pin="2"/>
 <pinref part="GND3" gate="1" pin="GND"/>
-<wire x1="2.54" y1="91.44" x2="2.54" y2="88.9" width="0.1524" layer="91"/>
+<wire x1="2.54" y1="91.44" x2="2.54" y2="86.36" width="0.1524" layer="91"/>
 </segment>
 <segment>
@@
 <pinref part="GND4" gate="1" pin="GND"/>
 <wire x1="-15.24" y1="96.52" x2="-15.24" y2="86.36" width="0.1524" layer="91"/>
+</segment>
+<segment>
+<pinref part="JP7" gate="G$1" pin="1"/>
+<wire x1="-50.8" y1="109.22" x2="-50.8" y2="88.9" width="0.1524" layer="91"/>
+<pinref part="C3" gate="G$1" pin="2"/>
+<wire x1="-35.56" y1="91.44" x2="-35.56" y2="88.9" width="0.1524" layer="91"/>
+<wire x1="-35.56" y1="88.9" x2="-35.56" y2="86.36" width="0.1524" layer="91"/>
+<wire x1="-50.8" y1="88.9" x2="-35.56" y2="88.9" width="0.1524" layer="91"/>
+<junction x="-35.56" y="88.9"/>
+<pinref part="GND2" gate="1" pin="GND"/>
+</segment>
+<segment>
+<pinref part="U2" gate="G$1" pin="VSS"/>
+<wire x1="106.68" y1="-20.32" x2="106.68" y2="-33.02" width="0.1524" layer="91"/>
+<pinref part="GND12" gate="1" pin="GND"/>
 </segment>
 </net>
@@
 </segment>
 </net>
-<net name="N$1" class="0">
-<segment>
-<pinref part="JP7" gate="G$1" pin="1"/>
-<wire x1="-50.8" y1="109.22" x2="-50.8" y2="88.9" width="0.1524" layer="91"/>
-<pinref part="C3" gate="G$1" pin="2"/>
-<pinref part="GND2" gate="1" pin="GND"/>
-<wire x1="-35.56" y1="91.44" x2="-35.56" y2="88.9" width="0.1524" layer="91"/>
-<wire x1="-35.56" y1="88.9" x2="-35.56" y2="86.36" width="0.1524" layer="91"/>
-<wire x1="-50.8" y1="88.9" x2="-35.56" y2="88.9" width="0.1524" layer="91"/>
-<junction x="-35.56" y="88.9"/>
-</segment>
-</net>
 <net name="+3V3" class="0">
 <segment>
@@
 </segment>
 </net>
-<net name="VSS" class="0">
-<segment>
-<pinref part="U2" gate="G$1" pin="VSS"/>
-<pinref part="GND14" gate="1" pin="GND"/>
-<wire x1="106.68" y1="-20.32" x2="106.68" y2="-30.48" width="0.1524" layer="91"/>
-</segment>
-</net>
